Commit message: Fixed naming issues

File: mirv_description/urdf/all_sensors.urdf.xacro (robot description, xacro)
@@ -5,20 +5,20 @@
                          	Cameras
      ========================================================= -->
-	<xacro:include filename="$(find road_robot_description)/urdf/cameras/camera_sensors.urdf.xacro" />
+	<xacro:include filename="$(find mirv_description)/urdf/cameras/camera_sensors.urdf.xacro" />
 	<!-- ====================================================
 						GPS
 	========================================================= -->
-	<xacro:include filename="$(find road_robot_description)/urdf/gps/gps_sensors.urdf.xacro" />
+	<xacro:include filename="$(find mirv_description)/urdf/gps/gps_sensors.urdf.xacro" />
 	<!-- ====================================================
                          	LiDAR
      ========================================================= -->
-	<xacro:include filename="$(find road_robot_description)/urdf/lidars/lidar_sensors.urdf.xacro" />
+	<xacro:include filename="$(find mirv_description)/urdf/lidars/lidar_sensors.urdf.xacro" />
 	<!-- ====================================================
                          	Motion
      ========================================================= -->
-	<xacro:include filename="$(find road_robot_description)/urdf/motion/motion_sensors.urdf.xacro" />
+	<xacro:include filename="$(find mirv_description)/urdf/motion/motion_sensors.urdf.xacro" />
 	<!-- ====================================================
                          	Misc
      ========================================================= -->
-	<xacro:include filename="$(find road_robot_description)/urdf/misc/misc_sensors.urdf.xacro" />
+	<xacro:include filename="$(find mirv_description)/urdf/misc/misc_sensors.urdf.xacro" />
 </robot>

File: mirv_description/urdf/cameras/camera_sensors.urdf.xacro (robot description, xacro)
@@ -5,27 +5,27 @@
      ========================================================= -->
 	<!-- Axis p5512 -->
-	<xacro:include filename="$(find road_robot_description)/urdf/cameras/rgb/axis_p5512.urdf.xacro" />
+	<xacro:include filename="$(find mirv_description)/urdf/cameras/rgb/axis_p5512.urdf.xacro" />
 	<!-- Axis m5013 -->
-	<xacro:include filename="$(find road_robot_description)/urdf/cameras/rgb/axis_m5013.urdf.xacro" />
+	<xacro:include filename="$(find mirv_description)/urdf/cameras/rgb/axis_m5013.urdf.xacro" />
 	<!-- uEye CP Gige -->
-	<xacro:include filename="$(find road_robot_description)/urdf/cameras/rgb/ueye_cp_gige.urdf.xacro" />
+	<xacro:include filename="$(find mirv_description)/urdf/cameras/rgb/ueye_cp_gige.urdf.xacro" />
 	<!-- ELP USB Camera w/ Normal Lens -->
-	<xacro:include filename="$(find road_robot_description)/urdf/cameras/rgb/elp_usb_camera.urdf.xacro" />
+	<xacro:include filename="$(find mirv_description)/urdf/cameras/rgb/elp_usb_camera.urdf.xacro" />
 	<!-- ====================================================
                          	RGBD
      ========================================================= -->
 	<!-- Asus Xtion PRO -->
-	<xacro:include filename="$(find road_robot_description)/urdf/cameras/rgbd/asus_xtion_pro.urdf.xacro" />
+	<xacro:include filename="$(find mirv_description)/urdf/cameras/rgbd/asus_xtion_pro.urdf.xacro" />
 	<!-- Kinect -->
-	<xacro:include filename="$(find road_robot_description)/urdf/cameras/rgbd/kinect.urdf.xacro" />
+	<xacro:include filename="$(find mirv_description)/urdf/cameras/rgbd/kinect.urdf.xacro" />
 	<!-- KinectV2 -->
-	<xacro:include filename="$(find road_robot_description)/urdf/cameras/rgbd/kinectv2.urdf.xacro" />
+	<xacro:include filename="$(find mirv_description)/urdf/cameras/rgbd/kinectv2.urdf.xacro" />
 	<!-- Orbbec Astra -->
-	<xacro:include filename="$(find road_robot_description)/urdf/cameras/rgbd/orbbec_astra.urdf.xacro" />
+	<xacro:include filename="$(find mirv_description)/urdf/cameras/rgbd/orbbec_astra.urdf.xacro" />
 	<!-- Fotonic E Series -->
-	<xacro:include filename="$(find road_robot_description)/urdf/cameras/rgbd/fotonic_e.urdf.xacro" />
+	<xacro:include filename="$(find mirv_description)/urdf/cameras/rgbd/fotonic_e.urdf.xacro" />
 	<!-- Intel Realsense R200 -->
-	<xacro:include filename="$(find road_robot_description)/urdf/cameras/rgbd/realsense_r200.urdf.xacro" />
+	<xacro:include filename="$(find mirv_description)/urdf/cameras/rgbd/realsense_r200.urdf.xacro" />
 	<!-- Intel Realsense D415 -->
-	<xacro:include filename="$(find road_robot_description)/urdf/cameras/rgbd/realsense_d415.urdf.xacro" />
+	<xacro:include filename="$(find mirv_description)/urdf/cameras/rgbd/realsense_d415.urdf.xacro" />
 </robot>

File: mirv_description/urdf/cameras/rgb/axis_m5013.urdf.xacro (robot description, xacro)
@@ -1,5 +1,5 @@
 <?xml version="1.0"?>
 <robot xmlns:xacro="http://ros.org/wiki/xacro" name="sensor_axis_m5013">
-     <xacro:include filename="$(find road_robot_description)/urdf/includes/materials.urdf.xacro"/>
+     <xacro:include filename="$(find mirv_description)/urdf/includes/materials.urdf.xacro"/>
      <xacro:property name="ptz_joint_effort_limit" value="100.0"/>
      <xacro:property name="ptz_joint_velocity_limit" value="100.0"/>
@@ -25,5 +25,5 @@
                     <origin xyz="0 0 0" rpy="0 ${M_PI/2} 0"/>
                     <geometry>
-                         <mesh filename="package://road_robot_description/meshes/cameras/axis/axis_m5013.dae" scale="1.0 1.0 1.0"/>
+                         <mesh filename="package://mirv_description/meshes/cameras/axis/axis_m5013.dae" scale="1.0 1.0 1.0"/>
                     </geometry>
                     <xacro:color_material color="${color}"/>
@@ -32,5 +32,5 @@
                     <origin xyz="0.0 0.0 0" rpy="0 ${M_PI/2} 0"/>
                     <geometry>
-                         <mesh filename="package://road_robot_description/meshes/cameras/axis/axis_m5013.stl" scale="1.0 1.0 1.0"/>
+                         <mesh filename="package://mirv_description/meshes/cameras/axis/axis_m5013.stl" scale="1.0 1.0 1.0"/>
                     </geometry>
                </collision>

File: mirv_description/urdf/cameras/rgb/axis_p5512.urdf.xacro (robot description, xacro)
@@ -1,5 +1,5 @@
 <?xml version="1.0"?>
 <robot xmlns:xacro="http://ros.org/wiki/xacro" name="sensor_axis_p5512">
-     <xacro:include filename="$(find road_robot_description)/urdf/includes/materials.urdf.xacro"/>
+     <xacro:include filename="$(find mirv_description)/urdf/includes/materials.urdf.xacro"/>
      <xacro:property name="ptz_joint_effort_limit" value="100.0"/>
      <xacro:property name="ptz_joint_velocity_limit" value="100.0"/>
@@ -25,5 +25,5 @@
                     <origin xyz="-0.3 0.0 -0.03" rpy="0 ${M_PI/2} 0"/>
                     <geometry>
-                         <mesh filename="package://road_robot_description/meshes/cameras/axis/axis_p5512.stl" scale="1.0 1.0 1.0"/>
+                         <mesh filename="package://mirv_description/meshes/cameras/axis/axis_p5512.stl" scale="1.0 1.0 1.0"/>
                     </geometry>
                     <xacro:color_material color="${color}"/>
@@ -33,5 +33,5 @@
                     <!-- because the origin of the mesh file is not at the "center" of the model-->
                     <geometry>
-                         <mesh filename="package://road_robot_description/meshes/cameras/axis/axis_p5512.stl" scale="1.0 1.0 1.0"/>
+                         <mesh filename="package://mirv_description/meshes/cameras/axis/axis_p5512.stl" scale="1.0 1.0 1.0"/>
                     </geometry>
                </collision>

File: mirv_description/urdf/cameras/rgb/elp_usb_camera.urdf.xacro (robot description, xacro)
@@ -1,5 +1,5 @@
 <?xml version="1.0"?>
 <robot xmlns:xacro="http://ros.org/wiki/xacro">
-     <xacro:include filename="$(find road_robot_description)/urdf/includes/materials.urdf.xacro"/>
+     <xacro:include filename="$(find mirv_description)/urdf/includes/materials.urdf.xacro"/>
      <xacro:macro name="sensor_elp_usb_cam" params="name parent *origin color">
           <joint name="${name}_joint" type="fixed">
@@ -19,5 +19,5 @@
                          <xacro:color_material color="${color}"/>
                          <geometry>
-                              <mesh filename="package://road_robot_description/meshes/cameras/misc/board_camera.dae" scale="1.0 1.0 1.0"/>
+                              <mesh filename="package://mirv_description/meshes/cameras/misc/board_camera.dae" scale="1.0 1.0 1.0"/>
                          </geometry>
                </visual>
@@ -25,5 +25,5 @@
                     <origin xyz="0.0 0.0 0.0" rpy="0 0 0"/>
                     <geometry>
-                         <mesh filename="package://road_robot_description/meshes/cameras/misc/board_camera.dae" scale="1.0 1.0 1.0"/>
+                         <mesh filename="package://mirv_description/meshes/cameras/misc/board_camera.dae" scale="1.0 1.0 1.0"/>
                     </geometry>
                </collision>

File: mirv_description/urdf/cameras/rgb/ueye_cp_gige.urdf.xacro (robot description, xacro)
@@ -1,5 +1,5 @@
 <?xml version="1.0"?>
 <robot xmlns:xacro="http://ros.org/wiki/xacro">
-     <xacro:include filename="$(find road_robot_description)/urdf/includes/materials.urdf.xacro"/>
+     <xacro:include filename="$(find mirv_description)/urdf/includes/materials.urdf.xacro"/>
      <xacro:macro name="sensor_ueye_cp_gige" params="name parent *origin color">
           <joint name="${name}_joint" type="fixed">
@@ -19,5 +19,5 @@
                          <xacro:color_material color="${color}"/>
                          <geometry>
-                              <mesh filename="package://road_robot_description/meshes/cameras/ids/ueye_cp_gige.stl" scale="1.0 1.0 1.0"/>
+                              <mesh filename="package://mirv_description/meshes/cameras/ids/ueye_cp_gige.stl" scale="1.0 1.0 1.0"/>
                          </geometry>
                </visual>
@@ -25,5 +25,5 @@
                     <origin xyz="0.0 0.0 0.0" rpy="0 0 0"/>
                     <geometry>
-                         <mesh filename="package://road_robot_description/meshes/cameras/ids/ueye_cp_gige.stl" scale="1.0 1.0 1.0"/>
+                         <mesh filename="package://mirv_description/meshes/cameras/ids/ueye_cp_gige.stl" scale="1.0 1.0 1.0"/>
                     </geometry>
                </collision>

File: mirv_description/urdf/cameras/rgbd/asus_xtion_pro.urdf.xacro (robot description, xacro)
@@ -1,5 +1,5 @@
 <?xml version="1.0"?>
 <robot name="sensor_asus_xtion_pro" xmlns:xacro="http://ros.org/wiki/xacro">
-     <xacro:include filename="$(find road_robot_description)/urdf/includes/materials.urdf.xacro"/>
+     <xacro:include filename="$(find mirv_description)/urdf/includes/materials.urdf.xacro"/>
      <xacro:property name="asus_xtion_scale" value="1.0"/>
      <xacro:property name="asus_xtion_pro_depth_rel_rgb_py" value="0.0270" />
@@ -40,5 +40,5 @@
                     <origin xyz="-0.01 0 0" rpy="${-M_PI/2} -${M_PI} ${-M_PI/2}"/>
                     <geometry>
-                         <mesh filename="package://road_robot_description/meshes/cameras/asus/asus_xtion_pro_live.dae" scale="${asus_xtion_scale} ${asus_xtion_scale} ${asus_xtion_scale}"/>
+                         <mesh filename="package://mirv_description/meshes/cameras/asus/asus_xtion_pro_live.dae" scale="${asus_xtion_scale} ${asus_xtion_scale} ${asus_xtion_scale}"/>
                     </geometry>
                     <xacro:color_material color="${color}"/>

File: mirv_description/urdf/cameras/rgbd/fotonic_e.urdf.xacro (robot description, xacro)
@@ -1,5 +1,5 @@
 <?xml version="1.0"?>
 <robot name="sensor_fotonic" xmlns:xacro="http://ros.org/wiki/xacro">
-	<xacro:include filename="$(find road_robot_description)/urdf/includes/materials.urdf.xacro"/>
+	<xacro:include filename="$(find mirv_description)/urdf/includes/materials.urdf.xacro"/>
 	<xacro:macro name="sensor_fotonic" params="name parent *origin color">
 		<joint name="${name}_joint" type="fixed">
@@ -18,5 +18,5 @@
 				<origin xyz="0.0 0.0 -0.04" rpy="0 0 0" /> <!-- to center the .dae model -->
 				<geometry>
-					<mesh filename= "package://road_robot_description/meshes/cameras/acroname/fotonic_e.stl" scale="1.0 1.0 1.0"/>
+					<mesh filename= "package://mirv_description/meshes/cameras/acroname/fotonic_e.stl" scale="1.0 1.0 1.0"/>
 				</geometry>
 				<xacro:color_material color="${color}"/>
@@ -25,5 +25,5 @@
 				<origin xyz="0.0 0 -0.04" rpy="0 0 0" />
 				<geometry>
-					<mesh filename= "package://road_robot_description/meshes/cameras/acroname/fotonic_e.stl" scale="1.0 1.0 1.0"/>
+					<mesh filename= "package://mirv_description/meshes/cameras/acroname/fotonic_e.stl" scale="1.0 1.0 1.0"/>
 				</geometry>
 			</collision>

File: mirv_description/urdf/cameras/rgbd/kinect.urdf.xacro (robot description, xacro)
@@ -1,5 +1,5 @@
 <?xml version="1.0"?>
 <robot name="sensor_kinect" xmlns:xacro="http://ros.org/wiki/xacro">
-	<xacro:include filename="$(find road_robot_description)/urdf/includes/materials.urdf.xacro"/>
+	<xacro:include filename="$(find mirv_description)/urdf/includes/materials.urdf.xacro"/>
 	<xacro:property name="M_PI" value="3.1415926535897931" />
 	<xacro:property name="cam_px" value="-0.087" />
@@ -43,5 +43,5 @@
 				<origin xyz="0 0 0" rpy="0 0 ${M_PI/2}"/>
 				<geometry>
-					<mesh filename="package://road_robot_description/meshes/cameras/microsoft/kinect.dae"/>
+					<mesh filename="package://mirv_description/meshes/cameras/microsoft/kinect.dae"/>
 				</geometry>
 				<xacro:color_material color="${color}"/>

File: mirv_description/urdf/cameras/rgbd/kinectv2.urdf.xacro (robot description, xacro)
@@ -1,5 +1,5 @@
 <?xml version="1.0"?>
 <robot name="sensor_kinectv2" xmlns:xacro="http://ros.org/wiki/xacro">
-     <xacro:include filename="$(find road_robot_description)/urdf/includes/materials.urdf.xacro"/>
+     <xacro:include filename="$(find mirv_description)/urdf/includes/materials.urdf.xacro"/>
      <xacro:property name="M_PI" value="3.1415926535897931" />
      <xacro:property name="cam_px" value="-0.087" />
@@ -49,8 +49,8 @@
                     <geometry>
                          <xacro:if value="${base}">
-                              <mesh filename="package://road_robot_description/meshes/cameras/microsoft/kinectv2.dae"/>
+                              <mesh filename="package://mirv_description/meshes/cameras/microsoft/kinectv2.dae"/>
                          </xacro:if>
                          <xacro:unless value="${base}">
-                              <mesh filename="package://road_robot_description/meshes/cameras/microsoft/kinectv2_nobase.dae"/>
+                              <mesh filename="package://mirv_description/meshes/cameras/microsoft/kinectv2_nobase.dae"/>
                          </xacro:unless>
                     </geometry>

File: mirv_description/urdf/cameras/rgbd/orbbec_astra.urdf.xacro (robot description, xacro)
@@ -1,5 +1,5 @@
 <?xml version="1.0"?>
 <robot name="sensor_orbbec_astra" xmlns:xacro="http://ros.org/wiki/xacro">
-     <xacro:include filename="$(find road_robot_description)/urdf/includes/materials.urdf.xacro"/>
+     <xacro:include filename="$(find mirv_description)/urdf/includes/materials.urdf.xacro"/>
      <xacro:property name="orbbec_astra_scale" value="1.0"/>
      <!-- RGB sensor - cam -->
@@ -46,5 +46,5 @@
                     <origin xyz="0 0 0" rpy="0 0 0"/>
                     <geometry>
-                         <mesh filename="package://road_robot_description/meshes/cameras/orbbec/orbbec_astra.dae" scale="${orbbec_astra_scale} ${orbbec_astra_scale} ${orbbec_astra_scale}"/>
+                         <mesh filename="package://mirv_description/meshes/cameras/orbbec/orbbec_astra.dae" scale="${orbbec_astra_scale} ${orbbec_astra_scale} ${orbbec_astra_scale}"/>
                     </geometry>
                     <xacro:color_material color="${color}"/>

File: mirv_description/urdf/cameras/rgbd/realsense_d415.urdf.xacro (robot description, xacro)
@@ -26,5 +26,5 @@
                     <origin xyz="${d415_cam_mount_from_center_offset} ${-d415_cam_depth_py} 0" rpy="${M_PI/2} 0 ${M_PI/2}"/>
                     <geometry>
-                         <mesh filename="package://road_robot_description/meshes/cameras/intel/realsense_d415.stl" />
+                         <mesh filename="package://mirv_description/meshes/cameras/intel/realsense_d415.stl" />
                     </geometry>
                     <material name="aluminum"/>

File: mirv_description/urdf/cameras/rgbd/realsense_r200.urdf.xacro (robot description, xacro)
@@ -7,5 +7,5 @@
                     <origin rpy="0 0 0" xyz="0 0 0"/>
                     <geometry>
-                         <mesh filename="package://road_robot_description/meshes/cameras/intel/realsense_r200.dae"/>
+                         <mesh filename="package://mirv_description/meshes/cameras/intel/realsense_r200.dae"/>
                     </geometry>
                </visual>

File: mirv_description/urdf/gps/gps_quad.urdf.xacro (robot description, xacro)
@@ -1,5 +1,5 @@
 <?xml version="1.0"?>
 <robot name="sensor_gps_quad" xmlns:xacro="http://ros.org/wiki/xacro">
-	<xacro:include filename="$(find road_robot_description)/urdf/includes/materials.urdf.xacro"/>
+	<xacro:include filename="$(find mirv_description)/urdf/includes/materials.urdf.xacro"/>
   	<xacro:macro name="sensor_gps_quad" params="name parent *origin color ref_lat ref_long ref_head drift vel_drift noise vel_noise update_rate">
 		<joint name="${name}_joint" type="revolute">
@@ -20,5 +20,5 @@
 				<origin rpy="0 0 0" xyz="0 0 0"/>
 				<geometry>
-					<mesh filename="package://road_robot_description/meshes/gps/antenna_3GO16.stl" scale="1.0 1.0 1.0"/>
+					<mesh filename="package://mirv_description/meshes/gps/antenna_3GO16.stl" scale="1.0 1.0 1.0"/>
 				</geometry>
 				<xacro:color_material color="${color}"/>

File: mirv_description/urdf/gps/gps_sensors.urdf.xacro (robot description, xacro)
@@ -4,7 +4,7 @@
                          	Misc
      ========================================================= -->
-	<xacro:include filename="$(find road_robot_description)/urdf/gps/gps_standard.urdf.xacro" />
-	<xacro:include filename="$(find road_robot_description)/urdf/gps/gps_quad.urdf.xacro" />
-	<xacro:include filename="$(find road_robot_description)/urdf/gps/gps_with_mast.urdf.xacro" />
-	<xacro:include filename="$(find road_robot_description)/urdf/gps/gps_with_dropout.urdf.xacro" />
+	<xacro:include filename="$(find mirv_description)/urdf/gps/gps_standard.urdf.xacro" />
+	<xacro:include filename="$(find mirv_description)/urdf/gps/gps_quad.urdf.xacro" />
+	<xacro:include filename="$(find mirv_description)/urdf/gps/gps_with_mast.urdf.xacro" />
+	<xacro:include filename="$(find mirv_description)/urdf/gps/gps_with_dropout.urdf.xacro" />
 </robot>

File: mirv_description/urdf/gps/gps_standard.urdf.xacro (robot description, xacro)
@@ -1,5 +1,5 @@
 <?xml version="1.0"?>
 <robot name="sensor_standard_gps" xmlns:xacro="http://ros.org/wiki/xacro">
-	<xacro:include filename="$(find road_robot_description)/urdf/includes/materials.urdf.xacro"/>
+	<xacro:include filename="$(find mirv_description)/urdf/includes/materials.urdf.xacro"/>
   	<xacro:macro name="sensor_standard_gps" params="name parent *origin color ref_lat ref_long ref_head drift vel_drift noise vel_noise update_rate">
 		<joint name="${name}_joint" type="fixed">
@@ -18,5 +18,5 @@
 				<origin rpy="0 0 0" xyz="0 0 0"/>
 				<geometry>
-					<mesh filename="package://road_robot_description/meshes/gps/antenna_3GO16.stl" scale="1.0 1.0 1.0"/>
+					<mesh filename="package://mirv_description/meshes/gps/antenna_3GO16.stl" scale="1.0 1.0 1.0"/>
 				</geometry>
 				<xacro:color_material color="${color}"/>
@@ -25,5 +25,5 @@
 				<origin rpy="0 0 0" xyz="0 0 0"/>
 				<geometry>
-					<mesh filename="package://road_robot_description/meshes/gps/antenna_3GO16.stl" scale="1.0 1.0 1.0"/>
+					<mesh filename="package://mirv_description/meshes/gps/antenna_3GO16.stl" scale="1.0 1.0 1.0"/>
 				</geometry>
 			</collision>

File: mirv_description/urdf/gps/gps_with_dropout.urdf.xacro (robot description, xacro)
@@ -1,5 +1,5 @@
 <?xml version="1.0"?>
 <robot name="sensor_gps_with_dropout" xmlns:xacro="http://ros.org/wiki/xacro">
-	<xacro:include filename="$(find road_robot_description)/urdf/includes/materials.urdf.xacro"/>
+	<xacro:include filename="$(find mirv_description)/urdf/includes/materials.urdf.xacro"/>
 	<!-- ====================================================
 						Helpers
@@ -52,5 +52,5 @@
 				<origin rpy="0 0 0" xyz="0 0 0"/>
 				<geometry>
-					<mesh filename="package://road_robot_description/meshes/gps/antenna_3GO16.stl" scale="1.0 1.0 1.0"/>
+					<mesh filename="package://mirv_description/meshes/gps/antenna_3GO16.stl" scale="1.0 1.0 1.0"/>
 				</geometry>
 				<xacro:color_material color="${color}"/>
@@ -59,5 +59,5 @@
 				<origin rpy="0 0 0" xyz="0 0 0"/>
 				<geometry>
-					<mesh filename="package://road_robot_description/meshes/gps/antenna_3GO16.stl" scale="1.0 1.0 1.0"/>
+					<mesh filename="package://mirv_description/meshes/gps/antenna_3GO16.stl" scale="1.0 1.0 1.0"/>
 				</geometry>
 			</collision>
@@ -69,6 +69,6 @@
 		<gazebo>
 			<plugin name="${name}_controller" filename="libgazebo_ros_gps_with_dropout.so">
-				<xacro:include filename="$(find road_robot_description)/config/gps/custom_gps_behavior.geofence"/>
-				<xacro:include filename="$(find road_robot_description)/config/gps/plots.xacro"/>
+				<xacro:include filename="$(find mirv_description)/config/gps/custom_gps_behavior.geofence"/>
+				<xacro:include filename="$(find mirv_description)/config/gps/plots.xacro"/>
 				<alwaysOn>1</alwaysOn>
 				<updateRate>${update_rate}</updateRate>
@@ -88,4 +88,4 @@
 		</gazebo>
 	</xacro:macro>
-	<!--<xacro:include filename="$(find road_robot_description)/config/gps/dropouts.xml"/>-->
+	<!--<xacro:include filename="$(find mirv_description)/config/gps/dropouts.xml"/>-->
 </robot>

File: mirv_description/urdf/gps/gps_with_mast.urdf.xacro (robot description, xacro)
@@ -46,5 +46,5 @@
                     <origin rpy="0 0 0" xyz="0 0 0"/>
                     <geometry>
-                         <mesh filename="package://road_robot_description/meshes/gps/antenna_3GO16.stl" scale="1.0 1.0 1.0"/>
+                         <mesh filename="package://mirv_description/meshes/gps/antenna_3GO16.stl" scale="1.0 1.0 1.0"/>
                     </geometry>
                     <xacro:color_material color="${color}"/>
@@ -53,5 +53,5 @@
                     <origin rpy="0 0 0" xyz="0 0 0"/>
                     <geometry>
-                         <mesh filename="package://road_robot_description/meshes/gps/antenna_3GO16.stl" scale="1.0 1.0 1.0"/>
+                         <mesh filename="package://mirv_description/meshes/gps/antenna_3GO16.stl" scale="1.0 1.0 1.0"/>
                     </geometry>
                </collision>
