Commit message: Fixed naming issues

File: mirv_description/urdf/lidars/hdl_32e.urdf.xacro (robot description, xacro)
@@ -18,5 +18,5 @@
       <visual>
         <geometry>
-          <mesh filename="package://road_robot_description/meshes/lidars/velodyne/HDL32E_base.dae" />
+          <mesh filename="package://mirv_description/meshes/lidars/velodyne/HDL32E_base.dae" />
         </geometry>
       </visual>
@@ -42,5 +42,5 @@
         <origin xyz="0 0 -0.09081" rpy="0 0 0" />
         <geometry>
-          <mesh filename="package://road_robot_description/meshes/lidars/velodyne/HDL32E_scan.dae" />
+          <mesh filename="package://mirv_description/meshes/lidars/velodyne/HDL32E_scan.dae" />
         </geometry>
       </visual>

File: mirv_description/urdf/lidars/hokuyo3d.urdf.xacro (robot description, xacro)
@@ -1,5 +1,5 @@
 <?xml version="1.0"?>
 <robot name="sensor_hokuyo3d" xmlns:xacro="http://ros.org/wiki/xacro">
-     <xacro:include filename="$(find road_robot_description)/urdf/includes/materials.urdf.xacro"/>
+     <xacro:include filename="$(find mirv_description)/urdf/includes/materials.urdf.xacro"/>
      <xacro:macro name="sensor_hokuyo3d" params="name visualize:=false parent *origin color">
           <joint name="${name}_fix_joint" type="fixed">
@@ -18,5 +18,5 @@
                     <origin xyz="0 0 0" rpy="0 0 0"/>
                     <geometry>
-                         <mesh filename="package://road_robot_description/meshes/lidars/hokuyo/hokuyo3d.stl"/>
+                         <mesh filename="package://mirv_description/meshes/lidars/hokuyo/hokuyo3d.stl"/>
                     </geometry>
                     <xacro:color_material color="${color}"/>
